File: KiCad/8088-FE2010A-SBC.sch (KiCad schematic (older format))
At the start: 61 parts, among them P1 KEYBOARD, P2 SPEAKER, P3 RESET, Q1 PN2222A, SW1 RESET, SW2 CONFIG, U1 8088, U10 74ALS245, U11 74ALS245, U12 74ALS244, U13 74ALS244, U14 74ALS04, U15 PIC12F629, U2 8087, U3 FE2010A, U4 28C256, U5 AS6C4008, U6 AS6C1008, U7 74LS573, U8 74LS573, X1 28.63636MHz

Commit message: Add 1.1 files
Signed-off-by: Sergey Kiselev <sergey.kiselev@intel.com>
Parts:
- removed JP1: ROM_1, my_components:Conn_Pin_Header_3x1_2.54mm, symbol CONN_01X03
- removed JP2: ROM_27, my_components:Conn_Pin_Header_3x1_2.54mm, symbol CONN_01X03
- removed SW2: CONFIG, my_components:IC_DIP8_300, symbol Switch_DIP-8
- removed U14: 74ALS04, my_components:IC_DIP14_300, symbol 74LS04
- removed U4: 28C256, my_components:IC_DIP28_600, symbol 28C256
- removed U6: AS6C1008, my_components:IC_DIP32_600, symbol AS6C1008
- added C17, C9: 0.1uF, my_components:Cap_Cer_508, symbol C
- added F1: 1.1A, my_components:Cap_Cer_508, symbol F_Small
- added JP1: ROM_A16, my_components:Conn_Pin_Header_2x1_2.54mm_NoKey, symbol JUMPER
- added JP2: XSEL, my_components:Conn_Pin_Header_2x1_2.54mm_NoKey, symbol JUMPER
- added JP3: RAMCS, my_components:Conn_Pin_Header_2x1_2.54mm_NoKey, symbol JUMPER
- added JP4: ROMCS, my_components:Conn_Pin_Header_2x1_2.54mm_NoKey, symbol JUMPER
- added R7: 10k, my_components:Res_762, symbol R
- added RR5: 10k, my_components:Conn_SIL6, symbol RR5
- added SW2: CONFIG, my_components:Switch_DIP_3_Positions, symbol Switch_DIP_3_Positions
- added SW3: UMB, my_components:Switch_DIP_5_Positions, symbol Switch_DIP_5_Positions
- added U14: 74F00, my_components:IC_DIP14_300, symbol 74LS00
- added U16: ATF16V8B, my_components:IC_DIP20_300, symbol ATF16V8B
- added U4: SST39SF010A, my_components:IC_DIP32_600, symbol SST39SF010A
- added U6: AS6C4008, my_components:IC_DIP32_600, symbol AS6C4008
- added U9: 74F573, my_components:IC_DIP20_300, symbol 74LS573
- U10, U11: value 74ALS245 -> 74F245
- U12, U13: value 74ALS244 -> 74F244
- U7, U8: value 74LS573 -> 74F573
- renumbered C17 to C18, C18 to C19, C19 to C20, C20 to C21, C21 to C22, C22 to C23, R7 to R8
Connections:
- net A0: now also U7.19 (O0), U4.12 (A0), U6.12 (A0); no longer U7.12 (O7)
- net A1: now also U7.18 (O1), U4.11 (A1), U6.11 (A1); no longer U7.13 (O6)
- net A10: now also U8.17 (O2), U4.23 (A10), U6.23 (A10); no longer U12.7 (Y2)
- net A11: now also U8.16 (O3), U4.25 (A11), U6.25 (A11); no longer U12.9 (Y1)
- net A12: now also U8.15 (O4), U4.4 (A12), U6.4 (A12); no longer U8.12 (O7)
- net A13: now also U8.14 (O5), U4.28 (A13), U6.28 (A13); no longer U8.13 (O6)
- net A14: now also U8.13 (O6), U4.29 (A14), U6.3 (A14); no longer U8.14 (O5)
- net A15: now also U8.12 (O7), U16.9 (I8), U4.3 (A15), U6.31 (A15); no longer U8.15 (O4)
- net A16: now also U16.5 (I4), U6.2 (A16), U9.15 (O4); no longer U8.16 (O3)
- net A17: now also U16.6 (I5), U6.30 (A17), U9.14 (O5); no longer U8.17 (O2)
- net A18: now also U16.7 (I6), U6.1 (A18), U9.13 (O6); no longer U8.18 (O1)
- net A19: now also U14.5, U16.8 (I7), U9.12 (O7); no longer U8.19 (O0)
- net A2: now also U7.17 (O2), U4.10 (A2), U6.10 (A2); no longer U7.14 (O5)
- net A3: now also U7.16 (O3), U4.9 (A3), U6.9 (A3); no longer U7.15 (O4)
- net A4: now also U7.15 (O4), U4.8 (A4), U6.8 (A4); no longer U7.16 (O3)
- net A5: now also U7.14 (O5), U4.7 (A5), U6.7 (A5); no longer U7.17 (O2)
- net A6: now also U7.13 (O6), U4.6 (A6), U6.6 (A6); no longer U7.18 (O1)
- net A7: now also U7.12 (O7), U4.5 (A7), U6.5 (A7); no longer U7.19 (O0)
- net A8: now also U8.19 (O0), U4.27 (A8), U6.27 (A8); no longer U12.3 (Y4)
- net A9: now also U8.18 (O1), U4.26 (A9), U6.26 (A9); no longer U12.5 (Y3)
- net AA10: now also U8.4 (D2); no longer U12.13 (A2)
- net AA11: now also U8.5 (D3); no longer U12.11 (A1)
- net AA12: now also U8.6 (D4); no longer U8.9 (D7)
- net AA13: now also U8.7 (D5); no longer U8.8 (D6)
- net AA14: now also U8.8 (D6); no longer U8.7 (D5)
- net AA15: now also U8.9 (D7); no longer U8.6 (D4)
- net AA16: now also U9.6 (D4); no longer U8.5 (D3)
- net AA17: now also U9.7 (D5); no longer U8.4 (D2)
- net AA18: now also U9.8 (D6); no longer U8.3 (D1)
- net AA19: now also U9.9 (D7); no longer U8.2 (D0)
- net AA8: now also U8.2 (D0); no longer U12.17 (A4)
- net AA9: now also U8.3 (D1); no longer U12.15 (A3)
- net AD0: now also U7.2 (D0), U4.13 (DQ0); no longer U7.9 (D7)
- net AD1: now also U7.3 (D1), U4.14 (DQ1); no longer U7.8 (D6)
- net AD2: now also U7.4 (D2), U4.15 (DQ2); no longer U7.7 (D5)
- net AD3: now also U7.5 (D3), U4.17 (DQ3); no longer U7.6 (D4)
- net AD4: now also U7.6 (D4), U4.18 (DQ4); no longer U7.5 (D3)
- net AD5: now also U7.7 (D5), U4.19 (DQ5); no longer U7.4 (D2)
- net AD6: now also U7.8 (D6), U4.20 (DQ6); no longer U7.3 (D1)
- net AD7: now also U7.9 (D7), U4.21 (DQ7); no longer U7.2 (D0)
- net ALE: now also U12.3 (Y4); no longer U12.18 (Y1)
- net AT_KBCLK: now also RR4.6; no longer RR4.5
- net AT_KBDATA: now also RR4.5; no longer RR4.4
- net CLK88: now also U12.8 (A4)
- net D3: now also U11.5 (A4); no longer U11.9 (A8)
- net D4: now also U11.6 (A5); no longer U11.8 (A7)
- net D6: now also U11.8 (A7); no longer U11.6 (A5)
- net D7: now also U11.9 (A8); no longer U11.5 (A4)
- net E0_PASS: now also RR4.4, SW2.4; no longer RR4.6
- net GND: now also U12.11 (A1), U12.13 (A2), C17.2, C9.2, JP2.1, R7.1, SW2.1, SW2.2, SW2.3, SW3.10, SW3.6, SW3.7, SW3.8, SW3.9, U14.10, U14.7 (GND), U14.7 (GND), U14.7 (GND), U14.7 (GND), U14.9, U16.10 (GND), U4.16 (GND), U6.16 (GND), U9.1 (~OE), U9.10 (GND), U9.2 (D0), U9.3 (D1), U9.4 (D2), U9.5 (D3); no longer P2.3 (P3)
- net KBCLK: now also RR1.8; no longer RR4.2
- net KBDATA: now also RR1.9; no longer RR4.3
- net LE: now also U9.11 (LE)
- net MD0: now also U6.13 (DQ0)
- net MD1: now also U6.14 (DQ1)
- net MD2: now also U6.15 (DQ2)
- net MD3: now also U11.15 (B4), U6.17 (DQ3); no longer U11.11 (B8)
- net MD4: now also U11.14 (B5), U6.18 (DQ4); no longer U11.12 (B7)
- net MD5: now also U6.19 (DQ5)
- net MD6: now also U11.12 (B7), U6.20 (DQ6); no longer U11.14 (B5)
- net MD7: now also U11.11 (B8), U6.21 (DQ7); no longer U11.15 (B4)
- net OSC: now also U12.2 (A1)
- net SPKR: now also U14.12, U14.13, U16.14 (I/O6)
- net VCC: now also C17.1, C9.1, F1.2, JP1.2, RR5.1 (COM), U14.14 (VCC), U14.14 (VCC), U14.14 (VCC), U14.14 (VCC), U16.20 (VCC), U4.32 (VCC), U6.32 (VCC), U9.20 (VCC); no longer P1.4 (P4)
- net XALE: now also U12.17 (A4); no longer U12.2 (A1)
- net XSEL: now also JP2.2
- net ~DACK0: now also U12.14 (Y3); no longer U12.12 (Y4)
- net ~DACK2: now also U12.5 (Y3); no longer U12.14 (Y3)
- net ~MEMR: now also U11.1 (DIR), U5.24 (~OE), U4.24 (~OE), U6.24 (~OE)
- net ~MEMW: now also U5.29 (~WE), U4.31 (~WE), U6.29 (~WE)
- net ~RAMCS: now also JP3.1; no longer U11.19 (~G)
- net ~ROMCS: now also JP4.2, U16.12 (I/O8), U4.22 (~CE); no longer U3.6 (~EPSL)
- net ~RQ/GT1: now also RR1.4; no longer RR1.3
- net ~RQ/GT2: now also RR1.3; no longer RR1.4
- net ~VID0: now also RR4.2, SW2.6; no longer RR1.8
- net ~VID1: now also RR4.3, SW2.5; no longer RR1.9
- net ~XDACK0: now also U12.6 (A3); no longer U12.8 (A4)
- net ~XDACK2: now also U12.15 (A3); no longer U12.6 (A3)
- net ~XMEMR: no longer U11.1 (DIR), U5.24 (~OE)
- net ~XMEMW: no longer U5.29 (~WE)
- net at R2.2: now also U12.12 (Y4)
- net at R3.2: now also U12.18 (Y1)
- net ~SPKR: now reaches R6.2
- net ~SPKR: now also U14.11, U16.15 (I/O5)
- new net: U14.3, U14.4
- new net: RR5.3, SW3.2, U16.17 (I/O3)
- new net: RR5.2, SW3.1, U16.18 (I/O2)
- new net: RR5.6, SW3.5, U16.2 (I1)
- new net: RR5.5, SW3.4, U16.3 (I2)
- new net: RR5.4, SW3.3, U16.4 (I3)
- new net KBD_VCC: F1.1, P1.4 (P4)
- new net ROM_A16: JP1.1, R7.2, U4.2 (A16)
- new net ~EPSL: JP4.1, U3.6 (~EPSL)
- new net ~RAMCS2: U14.6, U16.13 (I/O7), U6.22 (~CE)
- new net ~RAMENA: JP3.2, U11.19 (~G), U14.1, U14.2, U16.16 (I/O4)
- no-connect marks 19 -> 28
Other:
- note added: "SW3.1: C0000-C7FFF\nSW3.2: C8000-CFFFF\nSW3.3: D0000-D7FFF\nSW3.4: D8000-DFFFF\nSW3.5: E0000-EFFFF\n"
- note removed: "Pin 1\n----\nVCC\nVCC\nA14\n~WE"
- note removed: "Pin 27\n----\nVCC\nA14\n~WE\nA14"
- note removed: "ROM Type\n------\n27C128\n27C256\n28C256/SRAM\n29C256"
- moved on the sheet: C10, C11, C12, C13, C14, C15, C16, C18, C19, C20, C23, HOLE1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
